File: Reverse_Protection(COMPLETE)/element.brd (EAGLE design)
At the start: 100 x 80 mm, 3 parts

Commit message: update board
Parts:
- removed R2: 10k, adafruit:R0805
- added D1: BZX55, diode:DO35Z10
- FLIP: value IRFD9120 -> Si7145DP
Connections:
- net N$2: now also D1.A; no longer R2.2
- net N$3: now also D1.C; no longer R2.1
Changed lines of the file:
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@@
 </autorouter>
 <elements>
-<element name="FLIP" library="transistor-small-signal" library_urn="urn:adsk.eagle:library:401" package="C370-01" package3d_urn="urn:adsk.eagle:package:29750/1" value="IRFD9120" x="30.48" y="43.18"/>
-<element name="R1" library="adafruit" package="R0805" value="10k" x="33.02" y="25.4"/>
-<element name="R2" library="adafruit" package="R0805" value="10k" x="41.91" y="35.56" rot="R180"/>
+<element name="FLIP" library="transistor-small-signal" library_urn="urn:adsk.eagle:library:401" package="C370-01" package3d_urn="urn:adsk.eagle:package:29750/1" value="Si7145DP" x="30.48" y="43.18">
+<attribute name="MF" value="" x="30.48" y="43.18" size="1.778" layer="27" display="off"/>
+<attribute name="MPN" value="SI7145DP-T1-GE3" x="30.48" y="43.18" size="1.778" layer="27" display="off"/>
+<attribute name="OC_NEWARK" value="63R6006" x="30.48" y="43.18" size="1.778" layer="27" display="off"/>
+</element>
+<element name="R1" library="adafruit" package="R0805" value="10k" x="33.02" y="25.4">
+<attribute name="MF" value="" x="33.02" y="25.4" size="1.778" layer="27" display="off"/>
+<attribute name="MPN" value="RC0603FR-0710KL" x="33.02" y="25.4" size="1.778" layer="27" display="off"/>
+<attribute name="OC_NEWARK" value="68R0049" x="33.02" y="25.4" size="1.778" layer="27" display="off"/>
+</element>
+<element name="D1" library="diode" library_urn="urn:adsk.eagle:library:210" package="DO35Z10" package3d_urn="urn:adsk.eagle:package:43342/1" value="BZX55" x="24.13" y="31.75" rot="R270">
+<attribute name="MF" value="FAIRCHILD SEMICONDUCTOR" x="24.13" y="31.75" size="1.778" layer="27" rot="R270" display="off"/>
+<attribute name="MPN" value="BZX79C4V7" x="24.13" y="31.75" size="1.778" layer="27" rot="R270" display="off"/>
+<attribute name="OC_NEWARK" value="18C5987" x="24.13" y="31.75" size="1.778" layer="27" rot="R270" display="off"/>
+</element>
 </elements>
 <signals>
@@
 <contactref element="FLIP" pad="G"/>
 <contactref element="R1" pad="2"/>
-<contactref element="R2" pad="2"/>
-<wire x1="34.02" y1="25.4" x2="40.91" y2="35.56" width="0" layer="19" extent="1-1"/>
-<wire x1="34.29" y1="41.91" x2="34.02" y2="25.4" width="0" layer="19" extent="1-1"/>
+<contactref element="D1" pad="A"/>
+<wire x1="34.02" y1="25.4" x2="34.29" y2="41.91" width="0" layer="19" extent="1-1"/>
+<wire x1="24.13" y1="26.67" x2="34.02" y2="25.4" width="0" layer="19" extent="1-1"/>
 </signal>
 <signal name="N$3">
 <contactref element="FLIP" pad="S"/>
-<contactref element="R2" pad="1"/>
-<wire x1="42.91" y1="35.56" x2="34.29" y2="44.45" width="0" layer="19" extent="1-1"/>
+<contactref element="D1" pad="C"/>
+<wire x1="24.13" y1="36.83" x2="34.29" y2="44.45" width="0" layer="19" extent="1-1"/>
 </signal>
 </signals>

Commit message: update LTspice schematic
Parts:
- D1: value BZX55 -> 1N5250BTR
Changed lines of the file:
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@@
 <attribute name="OC_NEWARK" value="68R0049" x="33.02" y="25.4" size="1.778" layer="27" display="off"/>
 </element>
-<element name="D1" library="diode" library_urn="urn:adsk.eagle:library:210" package="DO35Z10" package3d_urn="urn:adsk.eagle:package:43342/1" value="BZX55" x="24.13" y="31.75" rot="R270">
+<element name="D1" library="diode" library_urn="urn:adsk.eagle:library:210" package="DO35Z10" package3d_urn="urn:adsk.eagle:package:43342/1" value="1N5250BTR" x="24.13" y="31.75" rot="R270">
 <attribute name="MF" value="FAIRCHILD SEMICONDUCTOR" x="24.13" y="31.75" size="1.778" layer="27" rot="R270" display="off"/>
 <attribute name="MPN" value="BZX79C4V7" x="24.13" y="31.75" size="1.778" layer="27" rot="R270" display="off"/>

Commit message: update schematic and board
Parts:
- removed D1: 1N5250BTR, diode:DO35Z10
- removed FLIP: Si7145DP, transistor-small-signal:C370-01
- added Q1: SI7145DP, Si7145DP:SO-8/PPAK/TEST
Connections:
- removed net N$1: FLIP.D, FLIP.D1
- removed net N$3: D1.C, FLIP.S
- new net IN: Q1.D@1, Q1.D@2, Q1.D@3, Q1.D@4, Q1.D@5
- new net OUT: Q1.S@1, Q1.S@2, Q1.S@3
- net N$2: now also Q1.G; no longer D1.A, FLIP.G
Routing:
- net N$2: track 0.00 -> 4.20 mm
- net OUT: track 0.00 -> 2.54 mm
Changed lines of the file:
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@@
 <setting verticaltext="up"/>
 </settings>
-<grid distance="50" unitdist="mil" unit="mil" style="lines" multiple="1" display="no" altdistance="5" altunitdist="mil" altunit="mil"/>
+<grid distance="50" unitdist="mil" unit="mil" style="lines" multiple="1" display="yes" altdistance="5" altunitdist="mil" altunit="mil"/>
 <layers>
 <layer number="1" name="Top" color="4" fill="1" visible="yes" active="yes"/>
@@
 <layer number="112" name="tSilk" color="7" fill="1" visible="no" active="yes"/>
 <layer number="113" name="ReferenceLS" color="7" fill="1" visible="no" active="no"/>
+<layer number="114" name="Badge_Outline" color="7" fill="1" visible="yes" active="yes"/>
+<layer number="115" name="ReferenceISLANDS" color="7" fill="1" visible="yes" active="yes"/>
 <layer number="116" name="Patch_BOT" color="9" fill="4" visible="no" active="yes"/>
 <layer number="118" name="Rect_Pads" color="7" fill="1" visible="no" active="no"/>
@@
 </autorouter>
 <elements>
-<element name="FLIP" library="transistor-small-signal" library_urn="urn:adsk.eagle:library:401" package="C370-01" package3d_urn="urn:adsk.eagle:package:29750/1" value="Si7145DP" x="30.48" y="43.18">
-<attribute name="MF" value="" x="30.48" y="43.18" size="1.778" layer="27" display="off"/>
-<attribute name="MPN" value="SI7145DP-T1-GE3" x="30.48" y="43.18" size="1.778" layer="27" display="off"/>
-<attribute name="OC_NEWARK" value="63R6006" x="30.48" y="43.18" size="1.778" layer="27" display="off"/>
-</element>
 <element name="R1" library="adafruit" package="R0805" value="10k" x="33.02" y="25.4">
 <attribute name="MF" value="" x="33.02" y="25.4" size="1.778" layer="27" display="off"/>
@@
 <attribute name="OC_NEWARK" value="68R0049" x="33.02" y="25.4" size="1.778" layer="27" display="off"/>
 </element>
-<element name="D1" library="diode" library_urn="urn:adsk.eagle:library:210" package="DO35Z10" package3d_urn="urn:adsk.eagle:package:43342/1" value="1N5250BTR" x="24.13" y="31.75" rot="R270">
-<attribute name="MF" value="FAIRCHILD SEMICONDUCTOR" x="24.13" y="31.75" size="1.778" layer="27" rot="R270" display="off"/>
-<attribute name="MPN" value="BZX79C4V7" x="24.13" y="31.75" size="1.778" layer="27" rot="R270" display="off"/>
-<attribute name="OC_NEWARK" value="18C5987" x="24.13" y="31.75" size="1.778" layer="27" rot="R270" display="off"/>
+<element name="Q1" library="Si7145DP" package="SO-8/PPAK/TEST" value="SI7145DP" x="40.894" y="27.305">
+<attribute name="MF" value="" x="40.894" y="27.305" size="1.778" layer="27" display="off"/>
+<attribute name="MPN" value="SI7145DP-T1-GE3" x="40.894" y="27.305" size="1.778" layer="27" display="off"/>
+<attribute name="OC_NEWARK" value="63R6006" x="40.894" y="27.305" size="1.778" layer="27" display="off"/>
 </element>
 </elements>
@@
 <contactref element="R1" pad="1"/>
 </signal>
-<signal name="N$1">
-<contactref element="FLIP" pad="D"/>
-<contactref element="FLIP" pad="D1"/>
-<wire x1="26.67" y1="41.91" x2="26.67" y2="44.45" width="0" layer="19" extent="1-1"/>
+<signal name="N$2">
+<contactref element="R1" pad="2"/>
+<contactref element="Q1" pad="G"/>
+<wire x1="34.02" y1="25.4" x2="38.224" y2="25.4" width="0.254" layer="1"/>
 </signal>
-<signal name="N$2">
-<contactref element="FLIP" pad="G"/>
-<contactref element="R1" pad="2"/>
-<contactref element="D1" pad="A"/>
-<wire x1="34.02" y1="25.4" x2="34.29" y2="41.91" width="0" layer="19" extent="1-1"/>
-<wire x1="24.13" y1="26.67" x2="34.02" y2="25.4" width="0" layer="19" extent="1-1"/>
+<signal name="IN">
+<contactref element="Q1" pad="D@5"/>
+<contactref element="Q1" pad="D@3"/>
+<contactref element="Q1" pad="D@1"/>
+<contactref element="Q1" pad="D@2"/>
+<contactref element="Q1" pad="D@4"/>
+<wire x1="43.689" y1="29.21" x2="43.689" y2="27.94" width="0" layer="19" extent="1-1"/>
+<wire x1="43.689" y1="26.67" x2="43.689" y2="27.94" width="0" layer="19" extent="1-1"/>
+<wire x1="43.689" y1="25.4" x2="43.689" y2="26.67" width="0" layer="19" extent="1-1"/>
+<wire x1="41.584" y1="27.305" x2="43.689" y2="27.94" width="0" layer="19" extent="1-1"/>
 </signal>
-<signal name="N$3">
-<contactref element="FLIP" pad="S"/>
-<contactref element="D1" pad="C"/>
-<wire x1="24.13" y1="36.83" x2="34.29" y2="44.45" width="0" layer="19" extent="1-1"/>
+<signal name="OUT">
+<contactref element="Q1" pad="S@2"/>
+<contactref element="Q1" pad="S@1"/>
+<contactref element="Q1" pad="S@3"/>
+<wire x1="38.224" y1="29.21" x2="38.224" y2="27.94" width="0.254" layer="1"/>
+<wire x1="38.224" y1="27.94" x2="38.224" y2="26.67" width="0.254" layer="1"/>
 </signal>
 </signals>
@@
 </board>
 </drawing>
-<compatibility>
-<note version="8.2" severity="warning">
-Since Version 8.2, EAGLE supports online libraries. The ids
-of those online libraries will not be understood (or retained)
-with this version.
-</note>
-<note version="8.3" severity="warning">
-Since Version 8.3, EAGLE supports URNs for individual library
-assets (packages, symbols, and devices). The URNs of those assets
-will not be understood (or retained) with this version.
-</note>
-<note version="8.3" severity="warning">
-Since Version 8.3, EAGLE supports the association of 3D packages
-with devices in libraries, schematics, and board files. Those 3D
-packages will not be understood (or retained) with this version.
-</note>
-</compatibility>
 </eagle>
